Commit message: basically working. Filter might go crazy when observation covariance is too small

File: nuturtle_description/urdf/diff_drive.urdf.xacro (robot description, xacro)
@@ -19,4 +19,10 @@
     <xacro:macro name="wheel" params="name color origin_xyz origin_rpy width radius">
      <link name="${name}">
+     <collision>
+         <origin xyz="${origin_xyz}" rpy="${origin_rpy}"/>
+         <geometry>
+            <cylinder length="${width}" radius="${radius}"/>
+        </geometry>
+     </collision>
        <visual>
          <origin xyz="${origin_xyz}" rpy="${origin_rpy}"/>
@@ -31,4 +37,10 @@
           </xacro:if>
        </visual>
+       <inertial>
+           <mass value="${diff_params['wheel_mass']}" />
+           <inertia ixx="${diff_params['wheel_mass']*(3*diff_params['wheel_radius']*diff_params['wheel_radius']+diff_params['wheel_width']*diff_params['wheel_width'])/12}" ixy="0.0" ixz="0.0"
+                iyy="${diff_params['wheel_mass']*(3*diff_params['wheel_radius']*diff_params['wheel_radius']+diff_params['wheel_width']*diff_params['wheel_width'])/12}" iyz="0.0"
+                izz="${diff_params['wheel_mass']*(diff_params['wheel_width']*diff_params['wheel_width'])/2}" />
+       </inertial>
      </link>
     </xacro:macro>
@@ -46,16 +58,42 @@
     <!--    link-->
     <link name="base_link">
-    <visual>
-     <origin xyz="${0.5*diff_params['chassis_length']-diff_params['wheel_width']} 0 ${0.5*diff_params['chassis_thickness']}" rpy="0 0 0"/>
-     <geometry>
-         <box size="${diff_params['chassis_length']} ${diff_params['wheel_base']-diff_params['wheel_width']} ${diff_params['chassis_thickness']}"/>
-      </geometry>
-        <xacro:insert_block name="pink_mat"/>
-    </visual>
+        <visual>
+        <origin xyz="0 0 0" rpy="0 0 0"/>
+         <geometry>
+             <box size="0.00001 0.00001 0.00001"/>
+          </geometry>
+        </visual>
+    </link>
+    <xacro:_joint name="base_link_chassis"
+      type="fixed"
+      origin_xyz ="0 0  ${diff_params['wheel_radius'] - diff_params['wheel_axle_offset']}" origin_rpy="0.0 0.0 0.0"
+      parent = "base_link"
+      child = "chassis"
+     axis = "1 0 0"/>
+    <link name="chassis">
+        <visual>
+             <origin xyz="${-1.0 * (0.5*diff_params['chassis_length']-diff_params['wheel_radius']) } 0 ${0.5*diff_params['chassis_thickness']}" rpy="0 0 0"/>
+         <geometry>
+             <box size="${diff_params['chassis_length']} ${diff_params['wheel_base']-diff_params['wheel_width']} ${diff_params['chassis_thickness']}"/>
+          </geometry>
+            <xacro:insert_block name="pink_mat"/>
+        </visual>
+        <collision>
+            <origin xyz="${-1.0 * (0.5*diff_params['chassis_length']-diff_params['wheel_radius']) } 0 ${0.5*diff_params['chassis_thickness']}" rpy="0 0 0"/>
+            <geometry>
+                <box size="${diff_params['chassis_length']} ${diff_params['wheel_base']-diff_params['wheel_width']} ${diff_params['chassis_thickness']}"/>
+            </geometry>
+        </collision>
+         <inertial>
+                <mass value="${diff_params['chassis_mass']}" />
+                <inertia ixx="${diff_params['chassis_mass']*((diff_params['wheel_base']-diff_params['wheel_width'])*(diff_params['wheel_base']-diff_params['wheel_width'])+diff_params['chassis_thickness']*diff_params['chassis_thickness'])/12}" ixy="0.0" ixz="0.0"
+                    iyy="${diff_params['chassis_mass']*(diff_params['chassis_length']*diff_params['chassis_length']+diff_params['chassis_thickness']*diff_params['chassis_thickness'])/12}" iyz="0.0"
+                    izz="${diff_params['chassis_mass']*((diff_params['wheel_base']-diff_params['wheel_width'])*(diff_params['wheel_base']-diff_params['wheel_width'])+diff_params['chassis_length']*diff_params['chassis_length'])/2}" />
+          </inertial>
     </link>
     <xacro:_joint name="left_wheel_axle"
            type="continuous"
-           origin_xyz = "0.0 ${0.5*diff_params['wheel_base']} 0.0" origin_rpy="0 0 0"
-           parent = "base_link"
+           origin_xyz = "0.0 ${0.5*diff_params['wheel_base']} ${diff_params['wheel_axle_offset']}" origin_rpy="0 0 0"
+           parent = "chassis"
            child = "left_wheel"
            axis = "0 1 0"/>
@@ -67,6 +105,6 @@
     <xacro:_joint name="right_wheel_axle"
         type="continuous"
-        origin_xyz = "0.0 ${-0.5*diff_params['wheel_base']} 0.0" origin_rpy="0.0 0.0 0.0"
-        parent = "base_link"
+        origin_xyz = "0.0 ${-0.5*diff_params['wheel_base']} ${diff_params['wheel_axle_offset']}" origin_rpy="0.0 0.0 0.0"
+        parent = "chassis"
         child = "right_wheel"
         axis = "0 1 0"/>
@@ -78,6 +116,6 @@
     <xacro:_joint name="base_link_ball_caster"
       type="fixed"
-      origin_xyz = "${diff_params['chassis_length']-1.5*diff_params['wheel_radius']} 0.0 ${-diff_params['wheel_radius']*0.5}" origin_rpy="0.0 0.0 0.0"
-      parent = "base_link"
+      origin_xyz = "${ -1 * (diff_params['chassis_length']-1.5*diff_params['wheel_radius'])} 0.0 ${(diff_params['wheel_radius']- diff_params['wheel_axle_offset'])*-0.5}" origin_rpy="0.0 0.0 0.0"
+      parent = "chassis"
       child = "ball_caster"
       axis = "0 1 0"/>
@@ -86,8 +124,25 @@
           <origin xyz="0 0 0" rpy="0 0 0"/>
           <geometry>
-              <sphere radius="${diff_params['wheel_radius']*0.5}"/>
+              <sphere radius="${(diff_params['wheel_radius']- diff_params['wheel_axle_offset'])*0.5}"/>
            </geometry>
              <xacro:insert_block name="pink_mat"/>
         </visual>
+          <collision>
+              <origin xyz="0 0 0" rpy="0 0 0"/>
+              <geometry>
+                <sphere radius="${(diff_params['wheel_radius']- diff_params['wheel_axle_offset'])*0.5}"/>
+              </geometry>
+          </collision>
       </link>
+      <xacro:_joint name="chassis_base_scan"
+        type="fixed"
+        origin_xyz = "0.0 0.0 ${diff_params['chassis_thickness']}" origin_rpy="0.0 0.0 0.0"
+        parent = "chassis"
+        child = "base_scan"
+        axis = "0 1 0"/>
+    <xacro:wheel name="base_scan"
+             color="yellow"
+             origin_xyz="0 0 ${diff_params['laser_scanner_height']/2}" origin_rpy="0 0 0"
+             width="${diff_params['laser_scanner_height']}"
+             radius="${diff_params['laser_scanner_radius']}"/>
 </robot>

Commit message: working!

File: nuturtle_description/urdf/diff_drive.urdf.xacro (robot description, xacro)
@@ -57,5 +57,5 @@
     </xacro:macro>
     <!--    link-->
-    <link name="base_link">
+    <link name="actual_robot">
         <visual>
         <origin xyz="0 0 0" rpy="0 0 0"/>

Commit message: clean up is done

File: nuturtle_description/urdf/diff_drive.urdf.xacro (robot description, xacro)
@@ -1,5 +1,5 @@
 <?xml version="1.0"?>
 <robot xmlns:xacro="http://www.ros.org/wiki/xacro" name="diff_drive">
-    <xacro:property name="diff_params" value="${load_yaml('$(find nuturtle_description)/config/diff_params.yaml')}" />
+    <xacro:property name="diff_params" value="${load_yaml('$(find real_world)/config/params.yaml')}" />
     <xacro:property name="grey_mat">
      <material name="arm_grey_mat">
